File: CDH-OBC/MCU.kicad_sch (KiCad schematic)
At the start: 1 part, among them U1 TMS5700714APZQQ1

Commit message: changes on rtc
Parts:
- U1: footprint OBC-Lib:PZ0100A_N -> PZ0100A_N
Changed lines of the file:
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@@
 			)
 		)
-		(property "Footprint" "OBC-Lib:PZ0100A_N"
+		(property "Footprint" "PZ0100A_N"
 			(at 179.07 74.93 0)
 			(hide yes)
@@
 			)
 		)
-		(property "Footprint" "OBC-Lib:PZ0100A_N"
+		(property "Footprint" "PZ0100A_N"
 			(at 82.55 157.48 0)
 			(hide yes)
@@
 			)
 		)
-		(property "Footprint" "OBC-Lib:PZ0100A_N"
+		(property "Footprint" "PZ0100A_N"
 			(at 77.47 68.58 0)
 			(hide yes)

Commit message: some progress on kicad
Parts:
- U1: footprint PZ0100A_N -> OBC-Lib:PZ0100A_N
Changed lines of the file:
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@@
 			)
 		)
-		(property "Footprint" "PZ0100A_N"
+		(property "Footprint" "OBC-Lib:PZ0100A_N"
 			(at 179.07 74.93 0)
 			(hide yes)
@@
 			)
 		)
-		(property "Footprint" "PZ0100A_N"
+		(property "Footprint" "OBC-Lib:PZ0100A_N"
 			(at 82.55 157.48 0)
 			(hide yes)
@@
 			)
 		)
-		(property "Footprint" "PZ0100A_N"
+		(property "Footprint" "OBC-Lib:PZ0100A_N"
 			(at 77.47 68.58 0)
 			(hide yes)
