File: CDH-OBC/MCU.kicad_sch (KiCad schematic)
At the start: 0 parts

Commit message: first inital changes
Parts:
- added U1: TMS5700714APZQQ1, PZ0100A_N, symbol OBC-lib:TMS5700714APZQQ1
Connections:
- new net Memory-IC[2A]: U1.67 (MIBSPI1_CLK)

Commit message: finished bulk of the schematic
Parts:
- added C28, C29, C30, C31, C32, C33, C34, C35, C36, C37, C38, C39, C40: 100nF, symbol Device:C_Small
- added J5: Conn_ARM_JTAG_SWD_20, symbol Connector:Conn_ARM_JTAG_SWD_20
- added J6: UART, symbol Connector_Generic:Conn_01x02
- added R35, R36, R37, R38: 33, symbol Device:R_Small_US
- added R39: 0, symbol Device:R_Small_US
- added TP10, TP11: TestPoint, symbol Connector:TestPoint
Connections:
- net GPIO0-*INT: now reaches U1.1 (GIOA[0]_INT[0])
- net GIOA7: now reaches U1.18 (GIOA[7]_INT[7])
- net BUCK_EN: now reaches U1.19 (N2HET1[0])
- net GPIO1-RST: now reaches U1.2 (GIOA[1]_INT[1])
- net CS2-SDA: now reaches U1.23 (SPI2_CS[0]_N)
- net AD1IN[0]: now reaches U1.42 (AD1IN[0])
- net AD1IN[1]: now reaches U1.49 (AD1IN[1])
- net GIOA2-WDI: now reaches U1.5 (GIOA[2]_INT[2])
- net AD1IN[2]: now reaches U1.51 (AD1IN[2])
- net AD1IN[3]: now reaches U1.52 (AD1IN[3])
- net AD1IN[4]: now reaches U1.54 (AD1IN[4])
- net MISO2-SDO: now reaches U1.69 (SPI2SOMI)
- net MOSI2-SDL: now reaches U1.70 (SPI2SIMO)
- net CLK2-SCL: now reaches U1.71 (SPI2CLK)
- net CS1(0)-CS#: now reaches U1.73 (MIBSPI1_CS[0]_N)
- net GPIO3-RESET: now reaches U1.8 (GIOA[3]_INT[3])
- net CS1(1)-CS#: now reaches U1.93 (MIBSPI1_CS[1]_N)
- net GND: now reaches U1.100 (VSS)
- net GND: now also U1.17 (VSS), U1.20 (VSS), U1.29 (VSS), U1.33 (VSS), U1.47 (VSSAD_ADREFLO), U1.59 (VSS), U1.7 (VSS), U1.72 (VSS), U1.86 (VSS), U1.87 (VSS), C28.1, C29.2, C30.2, C31.2, C32.2, C33.2, C34.2, C35.2, C36.2, C37.2, C38.2, C39.2, C40.2, J5.10 (GND), J5.12 (GND), J5.14 (GND), J5.16 (GND), J5.18 (GND), J5.20 (GND), J5.4 (GND), J5.6 (GND), J5.8 (GND), R39.2
- net +1V2: now reaches U1.13 (VCC)
- net +1V2: now also U1.21 (VCC), U1.30 (VCC), U1.32 (VCC), U1.61 (VCC), U1.88 (VCC), U1.99 (VCC), C34.1, C35.1, C36.1, C37.1, C38.1, C39.1, C40.1
- net Kelvin_GND: now reaches U1.15 (KELVIN_GND)
- net +3V3: now reaches U1.28 (VCCIO)
- net +3V3: now also U1.6 (VCCIO), U1.60 (VCCIO), U1.85 (VCCIO), U1.96 (VCCP), C28.2, C29.1, C30.1, C31.1, C32.1, C33.1, J5.1 (VTREF), J5.2 (VCC/NC)
- net ADREFHI: now reaches U1.46 (VCCAD_ADREFHI)
- net OSC_IN: now reaches U1.14 (OSCIN)
- net OSC_OUT: now reaches U1.16 (OSCOUT)
- net TEST: now reaches U1.24 (TEST)
- net at U1.3 (FLTP1): now also TP10.1
- net POR_NRESET: now reaches U1.31 (PORRST_N)
- net at U1.4 (FLTP2): now also TP11.1
- net CAN1TX: now reaches U1.62 (CAN1TX)
- net CAN1RX: now reaches U1.63 (CAN1RX)
- net MOSI1-SI: now reaches U1.65 (MIBSPI1_SIMO)
- net MISO1-SO: now reaches U1.66 (MIBSPI1_SOMI)
- net at U1.68 (MIBSPI1_ENA_N): now also R39.1
- net at U1.75 (TMS): now also J5.7 (TMS/SWDIO)
- net at U1.76 (TRST_N): now also J5.3 (~{TRST})
- net at U1.77 (TDI): now also R38.2
- net at U1.78 (TDO): now also R37.2
- net at U1.79 (TCK): now also R35.2
- net at U1.80 (RTCK): now also R36.2
- net MCU_RESET: now reaches U1.81 (RST_N)
- net MCU_RESET: now also J5.15 (~{SRST})
- net ~{ERROR}: now reaches U1.82 (ERROR_N)
- net CAN2TX: now reaches U1.91 (CAN2TX)
- net CAN2RX: now reaches U1.92 (CAN2RX)
- net at U1.94 (LINRX): now also J6.1 (Pin_1)
- net at U1.95 (LINTX): now also J6.2 (Pin_2)
- net Memory-IC[2A] renamed CLK1-SCK
- new net: J5.5 (TDI), R38.1
- new net: J5.13 (TDO/SWO), R37.1
- new net: J5.11 (RTCK), R36.1
- new net: J5.9 (TCK/SWCLK), R35.1
- no-connect marks 0 -> 14
Other:
- moved on the sheet: U1A, U1B

Commit message: finished schematic
Parts:
- added J7: Conn_02x15_Counter_Clockwise, Connector_PinHeader_2.54mm:PinHeader_2x15_P2.54mm_Vertical, symbol Connector_Generic:Conn_02x15_Counter_Clockwise
- C28, C29, C30, C31, C32, C33, C34, C35, C36, C37, C38, C39, C40: footprint (none) -> Capacitor_SMD:C_0603_1608Metric
- J5: footprint (none) -> Connector_PinHeader_2.54mm:PinHeader_2x10_P2.54mm_Vertical
- J6: footprint (none) -> Connector_PinHeader_2.54mm:PinHeader_1x02_P2.54mm_Vertical
- R35, R36, R37, R38, R39: footprint (none) -> Resistor_SMD:R_0603_1608Metric
- TP10, TP11: footprint (none) -> TestPoint:TestPoint_Pad_D1.0mm
Connections:
- net +1V2: now also J7.27 (Pin_27), J7.4 (Pin_4)
- net +3V3: now also J7.28 (Pin_28), J7.3 (Pin_3)
- net GND: now also J7.1 (Pin_1), J7.30 (Pin_30)
- net GIOA5: now reaches U1.10 (GIOA[5]_INT[5])
- net at U1.11 (N2HET1[22]): now also J7.25 (Pin_25)
- net GIOA6: now reaches U1.12 (GIOA[6]_INT[6])
- net at U1.22 (N2HET1[2]): now also J7.16 (Pin_16)
- net at U1.25 (N2HET1[4]): now also J7.17 (Pin_17)
- net at U1.26 (N2HET1[6]): now also J7.18 (Pin_18)
- net CS1(2)-CS#: now reaches U1.27 (MIBSPI1_CS[2]_N)
- net at U1.40 (AD1IN[16]): now also J7.12 (Pin_12)
- net at U1.41 (AD1IN[17]): now also J7.13 (Pin_13)
- net at U1.43 (AD1IN[7]): now also J7.7 (Pin_7)
- net at U1.44 (AD1IN[20]): now also J7.14 (Pin_14)
- net at U1.45 (AD1IN[21]): now also J7.15 (Pin_15)
- net at U1.48 (AD1IN[9]): now also J7.9 (Pin_9)
- net at U1.50 (AD1IN[10]): now also J7.10 (Pin_10)
- net at U1.53 (AD1IN[11]): now also J7.11 (Pin_11)
- net AD1IN[5]: now reaches U1.55 (AD1IN[5])
- net at U1.56 (AD1IN[6]): now also J7.6 (Pin_6)
- net at U1.57 (AD1IN[8]): now also J7.8 (Pin_8)
- net at U1.64 (N2HET1[24]): now also J7.26 (Pin_26)
- net at U1.74 (N2HET1[8]): now also J7.19 (Pin_19)
- net at U1.83 (N2HET1[10]): now also J7.20 (Pin_20)
- net at U1.89 (N2HET1[12]): now also J7.21 (Pin_21)
- net GIOA4: now reaches U1.9 (GIOA[4]_INT[4])
- net at U1.90 (N2HET1[14]): now also J7.22 (Pin_22)
- net at U1.97 (N2HET1[16]): now also J7.23 (Pin_23)
- net at U1.98 (N2HET1[18]): now also J7.24 (Pin_24)
- new net +5V: J7.2 (Pin_2), J7.29 (Pin_29)
- no-connect marks 14 -> 11
Other:
- moved on the sheet: C28, C29, C30, C31, C32, C33, C34, C35, C36, C37, C38, C39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
