File: CDH-OBC/Peripherals.kicad_sch (KiCad schematic)
At the start: 0 parts

Commit message: changes on mcu and cristal oscillator
Parts:
- added 1: 7M-16.000MAAJ-T, symbol OBC-lib:7M-16.000MAAJ-T
- added 11 (x2): TL3315NF250Q, symbol OBC-lib:TL3315NF250Q
- added C10, C15: 100nF, Capacitor_SMD:C_0603_1608Metric, symbol Device:C_Small
- added C11: 1uF, Capacitor_SMD:C_0603_1608Metric, symbol Device:C_Small
- added C12, C13: 22pF, Capacitor_SMD:C_0603_1608Metric, symbol Device:C_Small
- added C14: 4pF, Capacitor_SMD:C_0603_1608Metric, symbol Device:C_Small
- added R10: 100R, Resistor_SMD:R_0603_1608Metric, symbol Device:R_Small_US
- added R11, R9: 10k, Resistor_SMD:R_0603_1608Metric, symbol Device:R_Small_US
- added R12, R8: 1k, Resistor_SMD:R_0603_1608Metric, symbol Device:R_Small_US
- added R13: 0 ohm, Resistor_SMD:R_0603_1608Metric, symbol Device:R_Small_US
Connections:
- new net: 11.1, 11.2, R8.2
- new net: 11.3, 11.4, R10.1
- new net +3.3V: R8.1
- new net +3V3: R11.1
- new net GND: 1.2 (GND), 1.4 (GND), 11.1, 11.2, C10.1, C11.1, R12.2, R13.1, R9.2
- new net MicroController[1B]: 1.3, C11.2, C13.2, R10.2, R11.2, R12.1, R13.2
- new net MicroController[2B]: C12.1
- new net MicroController[3A]: 11.3, 11.4, C10.2, R9.1
- new net MicroController[3C]: C12.2, C13.1
Other:
- note added: "Cristal Oscillator"
- note added: "MCU reset"
