File: CDH-OBC/Peripherals.kicad_sch (KiCad schematic)
At the start: 0 parts

Commit message: finished bulk of the schematic
Parts:
- added C22, C41: 100nF, symbol Device:C_Small
- added C23: 1uF, symbol Device:C_Small
- added C26, C27: 22pF, symbol Device:C_Small
- added CR1: 7M-16.000MAAJ-T, CRYSTAL_TXC_7M, symbol OBC-lib:7M-16.000MAAJ-T
- added D7: LED, symbol Device:LED
- added R10, R8, R9: 100k, symbol Device:R_Small_US
- added R29, R33: 1k, symbol Device:R_Small_US
- added R30, R32: 10k, symbol Device:R_Small_US
- added R31: 100, symbol Device:R_Small_US
- added R34: 0, symbol Device:R_Small_US
- added SW4, SW5: SW_Push, symbol Switch:SW_Push
- added TH1, TH2, TH3: 100k (25C), symbol Device:Thermistor_US
- added TP5, TP6, TP7: TestPoint, symbol Connector:TestPoint
- added U6: TMP235A2DBZR, DBZ0003A-IPC_A, symbol OBC-lib:TMP235A2DBZR
Connections:
- new net: R29.1, SW4.1
- new net: D7.2 (A), R33.2
- new net: R31.1, SW5.2
- new net +3V3: C41.1, R10.1, R29.2, R32.1, R33.1, R8.1, R9.1, U6.1 (VDD)
- new net ADIN0: R8.2, TH1.1, TP5.1
- new net ADIN1: R9.2, TH2.1, TP6.1
- new net ADIN2: R10.2, TH3.1, TP7.1
- new net AIN1[4]: U6.2 (VOUT)
- new net GIOA7: C22.1, R30.1, SW4.2
- new net GND: C22.2, C23.2, C41.2, CR1.2, CR1.4, R30.2, R34.1, SW5.1, TH1.2, TH2.2, TH3.2, U6.3 (GND)
- new net Kelvin_GND: C26.2, C27.2
- new net MCU_RST: C23.1, R31.2, R32.2
- new net OSC_IN: C27.1, CR1.3
- new net OSC_OUT: C26.1, CR1.1
- new net TEST: R34.2
- new net ~{ERROR}: D7.1 (K)

Commit message: finished schematic
Parts:
- added R41: 100k, Resistor_SMD:R_0603_1608Metric, symbol Device:R_Small_US
- added TH4: 100k (25C), Resistor_SMD:R_0603_1608Metric, symbol Device:Thermistor_US
- added TP12: TestPoint, TestPoint:TestPoint_Pad_D1.0mm, symbol Connector:TestPoint
- C22, C23, C26, C27, C41: footprint (none) -> Capacitor_SMD:C_0603_1608Metric
- D7: footprint (none) -> LED_SMD:LED_0603_1608Metric
- R10, R29, R30, R31, R32, R33, R34, R8, R9, TH1, TH2, TH3: footprint (none) -> Resistor_SMD:R_0603_1608Metric
- TP5, TP6, TP7: footprint (none) -> TestPoint:TestPoint_Pad_D1.0mm
Connections:
- net +3V3: now also R41.1
- net GND: now also TH4.2
- new net ADIN3: R41.2, TH4.1, TP12.1

Commit message: finished adding footprints
Parts:
- SW4, SW5: footprint (none) -> OBC-Lib:SW_TL3315NF250Q
- U6: footprint DBZ0003A-IPC_A -> OBC-Lib:DBZ0003A-MFG
Changed lines of the file:
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@@
 			)
 		)
-		(property "Footprint" ""
+		(property "Footprint" "OBC-Lib:SW_TL3315NF250Q"
 			(at 46.99 45.72 0)
 			(hide yes)
@@
 			)
 		)
-		(property "Footprint" "DBZ0003A-IPC_A"
+		(property "Footprint" "OBC-Lib:DBZ0003A-MFG"
 			(at 220.98 38.1 0)
 			(hide yes)
@@
 			)
 		)
-		(property "Footprint" ""
+		(property "Footprint" "OBC-Lib:SW_TL3315NF250Q"
 			(at 41.91 78.74 0)
 			(hide yes)

Commit message: bulk schematic done
Parts:
- removed TP12, TP5, TP6, TP7: TestPoint, TestPoint:TestPoint_Pad_D1.0mm, symbol Connector:TestPoint
