File: CDH-OBC/CDH-OBC.kicad_sch (KiCad schematic)
At the start: 0 parts

Commit message: first inital changes
Other:
- added sheet Connectors (Connectors.kicad_sch)
- added sheet MCU peripherals (Peripherals.kicad_sch)
- added sheet Memory ICs (Memory.kicad_sch)
- added sheet Power (Power.kicad_sch)
- sheet MicroController ports: added Memory-IC[2A]; removed none
Changed lines of the file:
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@@
 		(comment 4 "Author: OCS division")
 	)
-	(sheet
-		(at 119.38 99.06)
+	(wire
+		(pts
+			(xy 111.76 55.88) (xy 111.76 49.53)
+		)
+		(stroke
+			(width 0)
+			(type default)
+		)
+	)
+	(wire
+		(pts
+			(xy 96.52 55.88) (xy 111.76 55.88)
+		)
+		(stroke
+			(width 0)
+			(type default)
+		)
+	)
+	(wire
+		(pts
+			(xy 111.76 49.53) (xy 115.57 49.53)
+		)
+		(stroke
+			(width 0)
+			(type default)
+		)
+	)
+	(sheet
+		(at 172.72 58.42)
+		(size 49.53 58.42)
+		(exclude_from_sim no)
+		(in_bom yes)
+		(on_board yes)
+		(dnp no)
+		(fields_autoplaced yes)
+		(stroke
+			(width 0.1524)
+			(type solid)
+		)
+		(fill
+			(color 0 0 0 0)
+		)
+		(property "Sheetname" "Memory ICs"
+			(at 172.72 57.7084 0)
+			(show_name no)
+			(do_not_autoplace no)
+			(effects
+				(font
+					(size 1.27 1.27)
+				)
+				(justify left bottom)
+			)
+		)
+		(property "Sheetfile" "Memory.kicad_sch"
+			(at 172.72 117.4246 0)
+			(show_name no)
+			(do_not_autoplace no)
+			(effects
+				(font
+					(size 1.27 1.27)
+				)
+				(justify left top)
+			)
+		)
+		(instances
+			(project "CDH-OBC"
+				(path "/c72b350f-acfc-44a2-bcbf-4f499b451c19"
+					(page "3")
+				)
+			)
+		)
+	)
+	(sheet
+		(at 133.35 39.37)
+		(size 46.99 12.7)
+		(exclude_from_sim no)
+		(in_bom yes)
+		(on_board yes)
+		(dnp no)
+		(fields_autoplaced yes)
+		(stroke
+			(width 0.1524)
+			(type solid)
+		)
+		(fill
+			(color 0 0 0 0)
+		)
+		(property "Sheetname" "MCU peripherals"
+			(at 133.35 38.6584 0)
+			(show_name no)
+			(do_not_autoplace no)
+			(effects
+				(font
+					(size 1.27 1.27)
+				)
+				(justify left bottom)
+			)
+		)
+		(property "Sheetfile" "Peripherals.kicad_sch"
+			(at 133.35 52.6546 0)
+			(show_name no)
+			(do_not_autoplace no)
+			(effects
+				(font
+					(size 1.27 1.27)
+				)
+				(justify left top)
+			)
+		)
+		(instances
+			(project "CDH-OBC"
+				(path "/c72b350f-acfc-44a2-bcbf-4f499b451c19"
+					(page "5")
+				)
+			)
+		)
+	)
+	(sheet
+		(at 52.07 140.97)
+		(size 20.32 38.1)
+		(exclude_from_sim no)
+		(in_bom yes)
+		(on_board yes)
+		(dnp no)
+		(fields_autoplaced yes)
+		(stroke
+			(width 0.1524)
+			(type solid)
+		)
+		(fill
+			(color 0 0 0 0)
+		)
+		(property "Sheetname" "Connectors"
+			(at 52.07 140.2584 0)
+			(show_name no)
+			(do_not_autoplace no)
+			(effects
+				(font
+					(size 1.27 1.27)
+				)
+				(justify left bottom)
+			)
+		)
+		(property "Sheetfile" "Connectors.kicad_sch"
+			(at 52.07 179.6546 0)
+			(show_name no)
+			(do_not_autoplace no)
+			(effects
+				(font
+					(size 1.27 1.27)
+				)
+				(justify left top)
+			)
+		)
+		(instances
+			(project "CDH-OBC"
+				(path "/c72b350f-acfc-44a2-bcbf-4f499b451c19"
+					(page "6")
+				)
+			)
+		)
+	)
+	(sheet
+		(at 87.63 104.14)
+		(size 29.21 44.45)
+		(exclude_from_sim no)
+		(in_bom yes)
+		(on_board yes)
+		(dnp no)
+		(fields_autoplaced yes)
+		(stroke
+			(width 0.1524)
+			(type solid)
+		)
+		(fill
+			(color 0 0 0 0)
+		)
+		(property "Sheetname" "Power"
+			(at 87.63 103.4284 0)
+			(show_name no)
+			(do_not_autoplace no)
+			(effects
+				(font
+					(size 1.27 1.27)
+				)
+				(justify left bottom)
+			)
+		)
+		(property "Sheetfile" "Power.kicad_sch"
+			(at 87.63 149.1746 0)
+			(show_name no)
+			(do_not_autoplace no)
+			(effects
+				(font
+					(size 1.27 1.27)
+				)
+				(justify left top)
+			)
+		)
+		(instances
+			(project "CDH-OBC"
+				(path "/c72b350f-acfc-44a2-bcbf-4f499b451c19"
+					(page "4")
+				)
+			)
+		)
+	)
+	(sheet
+		(at 66.04 44.45)
 		(size 30.48 44.45)
 		(exclude_from_sim no)
@@
 		)
 		(property "Sheetname" "MicroController"
-			(at 119.38 98.3484 0)
+			(at 66.04 43.7384 0)
 			(show_name no)
 			(do_not_autoplace no)
@@
 		)
 		(property "Sheetfile" "MCU.kicad_sch"
-			(at 119.38 144.0946 0)
-			(show_name no)
-			(do_not_autoplace no)
-			(effects
-				(font
-					(size 1.27 1.27)
-				)
-				(justify left top)
-			)
-		)
+			(at 66.04 89.4846 0)
+			(show_name no)
+			(do_not_autoplace no)
+			(effects
+				(font
+					(size 1.27 1.27)
+				)
+				(justify left top)
+			)
+		)
+		(pin "Memory-IC[2A]" input
+			(at 96.52 55.88 0)
+			(effects
+				(font
+					(size 1.27 1.27)
+				)
+				(justify right)
+			)
+		)

Commit message: finished bulk of the schematic
Other:
- removed sheet Connectors
- sheet MCU peripherals ports: added ADREFHI, GIOA7, Kelvin_GND, MCU_RST, OSC_IN, OSC_OUT, TEST, ~{ERROR}; removed none
- sheet Memory ICs ports: added ADIN0, ADIN1, ADIN2, CLK1-SCK, CLK2-SCL, CS1(0)-CS#, CS1(1)-CS, CS2-SDA, DCAN1RX, DCAN1TX, DCAN2RX, DCAN2TX, GIOA2-WDI, GPIO0-~{INT}, GPIO1-RESET, GPIO3-RESET, MISO1-SO, MISO2-SDO, MOSI1-SI, MOSI2-SDL, POR_NRESET, RTC_outV; removed none
- sheet Power ports: added BUCK_EN, VBAT_monitoring; removed none

Commit message: finished schematic
Other:
- sheet MCU peripherals ports: added ADIN0, ADIN1, ADIN2, ADIN3, AIN1[4]; removed ADREFHI
- sheet Memory ICs ports: added CS1(2)-#CS, GIOA4-LBK, GIOA5-LBK; removed ADIN0, ADIN1, ADIN2
- sheet MicroController ports: added AD1IN[0], AD1IN[1], AD1IN[2], AD1IN[3], AD1IN[4], AD1IN[5], ADREFHI, BUCK_EN, CAN1RX, CAN1TX, CAN2RX, CAN2TX, CLK1-SCK, CLK2-SCL, CS1(0)-CS#, CS1(1)-CS#, CS1(2)-CS#, CS2-SDA, GIOA2-WDI, GIOA4, GIOA5, GIOA6, GIOA7, GPIO0-*INT, GPIO1-RST, GPIO3-RESET, Kelvin_GND, MCU_RESET, MISO1-SO, MISO2-SDO, MOSI1-SI, MOSI2-SDL, OSC_IN, OSC_OUT, POR_NRESET, TEST, ~{ERROR}; removed Memory-IC[2A]
- sheet Power ports: added ADREFHI; removed none

Commit message: bulk schematic done
Changed lines of the file:
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@@
 		)
 		(pin "GIOA4-LBK" input
-			(at 153.67 72.39 0)
+			(at 153.67 74.93 0)
 			(effects
 				(font
@@
 		)
 		(pin "GIOA5-LBK" input
-			(at 153.67 74.93 0)
+			(at 153.67 72.39 0)
 			(effects
 				(font
