File: CDH-OBC/CDH-OBC.kicad_pcb (KiCad board)
At the start: 2 copper layers, 135 parts, among them J1 CAN1, J2 BAT, J3 CAN2, J4 Molex 6 pin, J5 Conn_ARM_JTAG_SWD_20, J6 UART, J7 Conn_02x15_Counter_Clockwise, Q1 PMOS, SW1 SW_Push, SW2 SW_Push, SW3 slide SW, SW4 SW_Push, SW5 SW_Push, U1 TMS5700714APZQQ1, U10 MCP1826S-1202E, U12 SN65HVD233, U13 SN65HVD233, U2 MR25H256AMDF, U3 TPS3850H50DRCR, U4 W25N02KVZEIR, U5 PCA2129T/Q900/2_51, U6 TMP235A2DBZR, U7 S25FL128LAGMFM010, U8 AP63205WU, U9 MIC37300-3.3WR

Commit message: bulk schematic done
Parts:
- removed J7: Conn_02x15_Counter_Clockwise, Connector_PinHeader_2.54mm:PinHeader_2x15_P2.54mm_Vertical
- removed R1: 10k, Resistor_SMD:R_0603_1608Metric
- removed TP12, TP2, TP3, TP4, TP5, TP6, TP7: TestPoint, TestPoint:TestPoint_Pad_D1.0mm
- added R42: 10k, Resistor_SMD:R_0603_1608Metric, F.Cu at (128.8, 93.4)
- added R43: 10k, Resistor_SMD:R_0603_1608Metric, F.Cu at (135.1, 94.4)
- added R44: 10k, Resistor_SMD:R_0603_1608Metric, F.Cu at (136.1, 104.9)
- added TP13: TestPoint, TestPoint:TestPoint_Pad_D1.0mm, F.Cu at (172.4, 113.4)
- C11, C21, C29, C30, C31, C32, C33, C34, C35, C36, C37, C38, C39, C40: moved to B.Cu
- moved J5 161.1 mm to (163.3, 138.7), turned to -90 degrees
- moved C28 159.2 mm to (165.9, 140.0), turned to -90 degrees
- moved C13 151.1 mm to (190.9, 109.7), turned to 180 degrees
- moved C14 151.1 mm to (189.2, 115.5), turned to 90 degrees
- moved C15 148.4 mm to (187.5, 115.5), turned to 90 degrees
- moved C16 145.9 mm to (187.5, 112.2), turned to -90 degrees
- moved R23 143.7 mm to (188.4, 118.7)
- moved R24 143.7 mm to (188.4, 121.2)
- moved R21 143.4 mm to (191.6, 107.0), turned to 90 degrees
- moved TH4 141.6 mm to (175.0, 102.4)
- moved R38 140.7 mm to (158.1, 135.2), turned to 90 degrees
- moved R22 140.6 mm to (190.9, 104.7), turned to 180 degrees
- moved R19 140.4 mm to (190.0, 107.0), turned to 90 degrees
- moved J4 139.9 mm to (187.0, 127.4), turned to -90 degrees
- moved C27 139.1 mm to (164.2, 100.9), turned to 90 degrees
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Connections:
- C14 pad 2: +5V -> Net-(U8-FB)
- C15 pad 2: +5V -> Net-(U8-FB)
- C19 pad 1: Net-(U9-VOUT) -> +3V3
- J4 pad 2: +5V -> +3V3
- J4 pad 3: +3V3 -> GND
- J4 pad 4: +3V3 -> +5V
- J4 pad 5: GND -> +3V3
- R23 pad 1: +5F -> +5V
- TP9 pad 1: Net-(U9-VOUT) -> +3V3
- U1 pad 10: /Memory ICs/GIOA5-LBK -> /Memory ICs/GIOA4-LBK
- U1 pad 9: /Memory ICs/GIOA4-LBK -> /Memory ICs/GIOA5-LBK
- U2 pad 2: /Memory ICs/MOSI1-SI -> /Memory ICs/MISO1-SO
- U2 pad 3: +3V3 -> Net-(U2-~{WP})
- U2 pad 5: /Memory ICs/MISO1-SO -> /Memory ICs/MOSI1-SI
- U2 pad 7: +3V3 -> Net-(U2-~{HOLD})
- U4 pad 3: Net-(U4-/HOLD_(IO3)) -> Net-(U4-/WP_(IO2))
- U8 pad 1: +5V -> Net-(U8-FB)
- U9 pad 3: Net-(U9-VOUT) -> +3V3
Routing:
- net /MCU peripherals/GIOA7: track 0.00 -> 89.7 mm, vias 0 -> 3
- net +3V3: track 0.00 -> 66.4 mm, vias 0 -> 31
- net /MCU peripherals/MCU_RST: track 0.00 -> 55.0 mm, vias 0 -> 2
- net /MicroController/AD1IN[5]: track 0.00 -> 53.2 mm, vias 0 -> 2
- net /Memory ICs/CAN2_P: track 0.00 -> 51.2 mm
- net /Memory ICs/CAN2_N: track 0.00 -> 50.4 mm
- net /MicroController/BUCK_EN: track 0.00 -> 48.3 mm, vias 0 -> 2
- net /Memory ICs/GPIO1-RESET: track 0.00 -> 45.9 mm, vias 0 -> 2
- net /Memory ICs/RTC_outV: track 0.00 -> 43.0 mm, vias 0 -> 2
- net +1V2: track 0.00 -> 42.2 mm, vias 0 -> 15
- net /Memory ICs/GPIO0-~{INT}: track 0.00 -> 39.1 mm, vias 0 -> 2
- net Net-(J5-~{TRST}): track 0.00 -> 38.9 mm, vias 0 -> 1
- net Net-(J5-TMS/SWDIO): track 0.00 -> 38.0 mm, vias 0 -> 1
- net /MCU peripherals/AIN1[4]: track 0.00 -> 38.0 mm, vias 0 -> 2
- net /MCU peripherals/ADIN3: track 0.00 -> 37.4 mm, vias 0 -> 2
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- added copper zone on In2.Cu, net +1V2
- added copper zone on In2.Cu, net +3V3
- added copper zone on F.Cu, net +5V
- added copper zone on In2.Cu, net +5V
- added copper zone on B.Cu, net GND
- added copper zone on F.Cu, net GND
- added copper zone on In1.Cu, net GND
- added copper zone on F.Cu, net Net-(Q1-S)
- added copper zone on F.Cu, net VBAT
- added copper zone on F.Cu, net VBUS
Other:
- board outline added: 86 x 86 mm
- copper layers 2 -> 4
- board text added: "{ "ViaStitching": "0.2", "stitch_zone_0": { "HSpacing": "1", "VSpacing": "1", "HOffset": "0", "VOffset": "0", "Clearance": "0", "Randomize": false } }"
- board text added: "{ "ViaStitching": "0.2", "stitch_zone_0": { "HSpacing": "3", "VSpacing": "3", "HOffset": "1.5", "VOffset": "0", "Clearance": "0", "Randomize": false } }"

Commit message: missed a trace
Routing:
- net Net-(D2-A): track 0.00 -> 1.52 mm
Changed lines of the file:
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@@
+	)
+	(segment
+		(start 193.7 76.19)
+		(end 193.7 74.67)
+		(width 0.2)
+		(layer "F.Cu")
+		(net "Net-(D2-A)")
 	)
 	(segment
